Commit message: Changed files so no urdf template is necessary. The urdf files exist with the corresponding sizes.

File: assets/urdf/cube0.urdf (robot description, URDF)
Before this commit: robot cube, 1 links, 0 joints
Links:
- link baseLink: mass 0.12 -> 0.8; geometry collision box size=0.08 0.08 0.08; visual box size=0.08 0.08 0.08

File: assets/urdf/cube1.urdf (robot description, URDF)
Before this commit: robot cube, 1 links, 0 joints
Links:
- link baseLink: mass 0.18 -> 0.7; geometry collision box size=0.07 0.07 0.07; visual box size=0.07 0.07 0.07

File: assets/urdf/cube2.urdf (robot description, URDF)
Before this commit: robot cube, 1 links, 0 joints
Links:
- link baseLink: mass 0.21000000000000002 -> 0.6; geometry collision box size=0.06 0.06 0.06; visual box size=0.06 0.06 0.06

File: assets/urdf/cube3.urdf (robot description, URDF)
Before this commit: robot cube, 1 links, 0 joints
Links:
- link baseLink: mass 0.15000000000000002 -> 0.5

File: assets/urdf/cube4.urdf (robot description, URDF)
Before this commit: robot cube, 1 links, 0 joints
Links:
- link baseLink: mass 0.24 -> 0.4; geometry collision box size=0.04 0.04 0.04; visual box size=0.04 0.04 0.04
